File: src/kicad/hrpi/hrpi.sch (KiCad schematic (older format))
At the start: 30 parts, among them P1 CONN_02X20, P10 CONN_01X01, P11 CONN_01X04, P12 CONN_01X05, P13 CONN_01X05, P14 CONN_01X05, P15 CONN_01X04, P16 CONN_01X04, P17 CONN_01X02, P2 CONN_02X04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

Commit message: BUGFIX
Parts:
- removed D?: LED, symbol LED
- removed R?: R, symbol R
- D5: renamed from D?; footprint (none) -> LEDs:LED-3MM
- R7: renamed from R?; footprint (none) -> Resistors_SMD:R_0805_HandSoldering
Connections:
- wire segments 131 -> 128
Changed lines of the file:
@@
 EESchema Schematic File Version 2
-LIBS:test-rescue
+LIBS:hrpi-rescue
 LIBS:power
 LIBS:device
@@
 LIBS:contrib
 LIBS:valves
-LIBS:test-cache
+LIBS:hrpi-cache
 EELAYER 25 0
 EELAYER END
@@
 OK
 $Comp
-L LED D?
-U 1 1 5769A7EA
-P 4750 1550
-F 0 "D?" H 4750 1650 50  0000 C CNN
-F 1 "LED" H 4750 1450 50  0000 C CNN
-F 2 "" H 4750 1550 50  0000 C CNN
-F 3 "" H 4750 1550 50  0000 C CNN
-	1    4750 1550
-	-1   0    0    1
-$EndComp
-$Comp
-L LED D?
+L LED D5
 U 1 1 5769A8C2
 P 4750 1700
-F 0 "D?" H 4750 1800 50  0000 C CNN
+F 0 "D5" H 4750 1800 50  0000 C CNN
 F 1 "LED" H 4750 1600 50  0000 C CNN
-F 2 "" H 4750 1700 50  0000 C CNN
+F 2 "LEDs:LED-3MM" H 4750 1700 50  0001 C CNN
 F 3 "" H 4750 1700 50  0000 C CNN
 	1    4750 1700
@@
 $EndComp
 Wire Wire Line
-	4550 1550 4250 1550
-Wire Wire Line
 	4550 1700 4250 1700
 Wire Wire Line
-	4950 1550 5350 1550
-Wire Wire Line
 	4950 1700 5350 1700
 $Comp
-L R R?
-U 1 1 5769C75A
-P 5500 1550
-F 0 "R?" V 5580 1550 50  0000 C CNN
-F 1 "R" V 5500 1550 50  0000 C CNN
-F 2 "" V 5430 1550 50  0000 C CNN
-F 3 "" H 5500 1550 50  0000 C CNN
-	1    5500 1550
-	0    1    1    0
-$EndComp
-$Comp
-L R R?
+L R R7
 U 1 1 5769C814
 P 5500 1700
-F 0 "R?" V 5580 1700 50  0000 C CNN
+F 0 "R7" V 5580 1700 50  0000 C CNN
 F 1 "R" V 5500 1700 50  0000 C CNN
-F 2 "" V 5430 1700 50  0000 C CNN
+F 2 "Resistors_SMD:R_0805_HandSoldering" V 5430 1700 50  0001 C CNN
 F 3 "" H 5500 1700 50  0000 C CNN
 	1    5500 1700
@@
 $EndComp
 Wire Wire Line
-	5650 1550 5650 1700
-Wire Wire Line
 	5650 1700 6000 1700
-Connection ~ 5650 1700
 Text Label 5800 1700 0    60   ~ 0
 GND
 Text Label 4300 1700 0    60   ~ 0
 RCOK
-Text Label 4300 1550 0    60   ~ 0
-OK
 $EndSCHEMATC
